File: Power/EEE3088F_2024_Group_52_Power.kicad_pcb (KiCad board)
At the start: 2 copper layers, 35 x 40 mm, 29 parts, among them J1 Conn_02x08_Odd_Even, J2 Conn_01x02, Q1 AO3401A, SW1 MINI MSK12CO2, U1 LMV321IDBVR, U2 TP4056, U3 DRV8837CDSGR, U4 DRV8837CDSGR

Commit message: Proposed fixes to power PCB flaws
Connections:
- Q1 pad 2: VCC -> BATT
- Q1 pad 3: BATT -> VCC
Routing:
- net VCC: track 92.5 -> 81.8 mm, vias 6 -> 5
- net BATT: track 51.5 -> 53.3 mm, vias 3 -> 4
Changed lines of the file:
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@@
 	)
 	(paper "A4")
+	(title_block
+		(title "EEE3088F_2024_Group_52_Power")
+		(date "2024-03-25")
+		(rev "v1")
+		(comment 3 "Triss Naidoo")
+		(comment 4 "NDXTRI021")
+	)
 	(layers
 		(0 "F.Cu" signal)
@@
 		(tags "capacitor")
 		(property "Reference" "C2"
-			(at 0 -1.43 270)
+			(at 0 -1.43 -90)
 			(layer "F.SilkS")
 			(effects
@@
 		)
 		(property "Value" "10u"
-			(at 0 1.43 270)
+			(at 0 1.43 -90)
 			(layer "F.Fab")
 			(effects
@@
 		)
 		(fp_text user "${REFERENCE}"
-			(at 0 0 270)
+			(at 0 0 -90)
 			(layer "F.Fab")
 			(effects
@@
 		(tags "solder jumper open")
 		(property "Reference" "JP2"
-			(at -1 -2 270)
+			(at -1 -2 -90)
 			(layer "F.SilkS")
 			(effects
@@
 		)
 		(property "Value" "Jumper_2_Open"
-			(at 0 1.9 270)
+			(at 0 1.9 -90)
 			(layer "F.Fab")
 			(effects
@@
 		)
 		(fp_text user "1"
-			(at -2.6 0 270)
+			(at -2.6 0 -90)
 			(layer "F.SilkS")
 			(effects
@@
 		)
 		(fp_text user "2"
-			(at 2.6 0 270)
+			(at 2.6 0 -90)
 			(layer "F.SilkS")
 			(effects
@@
 		(tags "resistor")
 		(property "Reference" "R1"
-			(at 0.1 -1.4 270)
+			(at 0.1 -1.4 -90)
 			(layer "F.SilkS")
 			(effects
@@
 		)
 		(property "Value" "1M"
-			(at 0 -1.4 270)
+			(at 0 -1.4 -90)
 			(layer "F.Fab")
 			(effects
@@
 		)
 		(fp_text user "${REFERENCE}"
-			(at 0 0 270)
+			(at 0 0 -90)
 			(layer "F.Fab")
 			(effects
@@
 			(size 1 0.8)
 			(layers "F.Cu" "F.Paste" "F.Mask")
-			(net 4 "VCC")
+			(net 15 "BATT")
 			(pinfunction "S")
 			(pintype "passive")
@@
 			(size 1 0.8)
 			(layers "F.Cu" "F.Paste" "F.Mask")
-			(net 15 "BATT")
+			(net 4 "VCC")
 			(pinfunction "D")
 			(pintype "passive")
@@
 		(tags "connector JST PH top entry")
 		(property "Reference" "J2"
-			(at 1 -2.55 360)
+			(at 1 -2.55 0)
 			(layer "F.SilkS")
 			(effects
@@
 		)
 		(property "Value" "Conn_01x02"
-			(at 1 7.45 360)
+			(at 1 7.45 0)
 			(layer "F.Fab")
 			(effects
@@
 		)
 		(fp_text user "${REFERENCE}"
-			(at 1 2.5 360)
+			(at 1 2.5 0)
 			(layer "F.Fab")
 			(effects
@@
 		(tags "Through hole pin header THT 2x08 2.54mm double row")
 		(property "Reference" "J1"
-			(at 1.27 2.33 270)
+			(at 1.27 2.33 -90)
 			(layer "B.SilkS")
 			(effects
@@
 		)
 		(property "Value" "Conn_02x08_Odd_Even"
-			(at 1.27 -20.11 270)
+			(at 1.27 -20.11 -90)
 			(layer "B.Fab")
 			(effects
@@
 		)
 		(fp_text user "${REFERENCE}"
-			(at 1.27 -8.89 360)
+			(at 1.27 -8.89 0)
 			(layer "B.Fab")
 			(effects
@@
 	)
 	(gr_line
+		(start 117.25 40)
+		(end 117.25 41.5)
+		(stroke
+			(width 0.2)
+			(type default)
+		)
+		(layer "F.Cu")
+		(net 4)
+	)
+	(gr_line
+		(start 133 50)
+		(end 134.5 49)
+		(stroke
+			(width 0.2)
+			(type default)
+		)
+		(layer "F.Cu")
+		(net 15)
+	)
+	(gr_line
+		(start 131 44.75)
+		(end 131 46.5)
+		(stroke
+			(width 0.2)
+			(type default)
+		)
+		(layer "F.Cu")
+		(net 4)
+	)
+	(gr_line
+		(start 117.25 41.5)
+		(end 119 43)
+		(stroke
+			(width 0.2)
+			(type default)
+		)
+		(layer "F.Cu")
+		(net 4)
+	)
+	(gr_line
+		(start 128.5 47.5)
+		(end 128.5 48.75)
+		(stroke
+			(width 0.2)
+			(type default)
+		)
+		(layer "F.Cu")
+		(net 15)
+	)
+	(gr_line
+		(start 128.5 48.75)
+		(end 129.5 50)
+		(stroke
+			(width 0.2)
+			(type default)
+		)
+		(layer "F.Cu")
+		(net 15)
+	)
+	(gr_line
+		(start 119 43)
+		(end 129 43)
+		(stroke
+			(width 0.2)
+			(type default)
+		)
+		(layer "F.Cu")
+		(net 4)
+	)
+	(gr_line
+		(start 129 43)
+		(end 131 44.75)
+		(stroke
+			(width 0.2)
+			(type default)
+		)
+		(layer "F.Cu")
+		(net 4)
+	)
+	(gr_line
+		(start 129.5 50)
+		(end 133 50)
+		(stroke
+			(width 0.2)
+			(type default)
+		)
+		(layer "F.Cu")
+		(net 15)
+	)
+	(gr_line
 		(start 111 17)
 		(end 144 17)
@@
 	)
 	(segment
-		(start 128.736 51.5)
-		(end 128.736 47.6)
-		(width 0.4)
-		(layer "F.Cu")
-		(net 4)
-	)
-	(segment
 		(start 132.15 21.4)
 		(end 131.75 21)
@@
 	)
 	(segment
-		(start 127.65 47.45)
-		(end 127.2 47)
-		(width 0.4)
-		(layer "F.Cu")
-		(net 4)
-	)
-	(segment
 		(start 137 19.275)
 		(end 134 19.275)
@@
 	)
 	(segment
-		(start 128.586 47.45)
-		(end 127.65 47.45)
-		(width 0.4)
-		(layer "F.Cu")
-		(net 4)
-	)
-	(segment
 		(start 116 19.225)
 		(end 119 19.225)
@@
 	)
 	(segment
-		(start 128.736 47.6)
-		(end 128.586 47.45)
+		(start 131 46.5)
+		(end 131.75 47.25)
 		(width 0.4)
 		(layer "F.Cu")
@@
 		(net 4)
 	)
-	(via
-		(at 130 42)
-		(size 0.6)
-		(drill 0.3)
-		(layers "F.Cu" "B.Cu")
+	(segment
+		(start 130.886 46.5)
+		(end 131 46.5)
+		(width 0.4)
+		(layer "F.Cu")
 		(net 4)
 	)
 	(via
-		(at 126.25 32.25)
+		(at 130 42)
 		(size 0.6)
 		(drill 0.3)
@@
 	)
 	(via
-		(at 127.2 47)
+		(at 126.25 32.25)
 		(size 0.6)
 		(drill 0.3)
@@
 	)
 	(segment
-		(start 127.2 44.8)
-		(end 127.2 47)
-		(width 0.4)
-		(layer "B.Cu")
-		(net 4)
-	)
-	(segment
 		(start 126.255 20.255)
 		(end 126.255 23.735)
@@
 	)
 	(segment
-		(start 127.2 44.8)
-		(end 130 42)
-		(width 0.4)
-		(layer "B.Cu")
-		(net 4)
-	)
-	(segment
 		(start 132.5 21.4)
 		(end 128.59 21.4)
@@
 	)
 	(segment
-		(start 131.75 48.25)
-		(end 131.75 47.25)
+		(start 127.2 47)
+		(end 127.65 47.45)
 		(width 0.4)
 		(layer "F.Cu")
@@
 	)
 	(segment
+		(start 128.586 47.45)
+		(end 127.65 47.45)
+		(width 0.4)
+		(layer "F.Cu")
+		(net 15)
+	)
+	(segment
 		(start 143 36.68)
 		(end 141 34.68)
@@
 	)
 	(segment
-		(start 131 46.5)
-		(end 131.75 47.25)
+		(start 128.736 47.6)
+		(end 128.586 47.45)
 		(width 0.4)
 		(layer "F.Cu")
@@
 	)
 	(segment
-		(start 130.886 46.5)
-		(end 131 46.5)
-		(width 0.4)
-		(layer "F.Cu")
-		(net 15)
-	)
-	(segment
 		(start 113.95 44.75)
 		(end 113.95 46.85)
@@
 	)
 	(via
+		(at 127.2 47)
+		(size 0.6)
+		(drill 0.3)
+		(layers "F.Cu" "B.Cu")
+		(net 15)
+	)
+	(via
 		(at 131.1 48.9)
 		(size 0.6)
@@
 		(net 15)
 	)
+	(segment
+		(start 127.2 44.8)
+		(end 127.2 47)
+		(width 0.4)
+		(layer "B.Cu")
+		(net 15)
+	)
